Commit message: Added Bracelet Camera

File: voaige_description/arms/kinova_gen3/urdf/GEN3-6DOF_VISION_URDF_ARM_V01.urdf (robot description, URDF)
Before this commit: robot mk1, 7 links, 6 joints
Links:
- link base_link: geometry collision mesh filename=package://voaige_description/arms/kinova_gen3/meshes/base_l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; visual mesh filename=package://voaige_description/arms/kinova_gen3/meshes/base_l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
- link bicep_link: geometry collision mesh filename=package://voaige_description/arms/kinova_gen3/meshes/bicep_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; visual mesh filename=package://voaige_description/arms/kinova_gen3/meshes/bicep_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
- link bracelet_link: geometry collision mesh filename=package://voaige_description/arms/kinova_gen3/meshes/bracel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; visual mesh filename=package://voaige_description/arms/kinova_gen3/meshes/bracel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
- link forearm_link: geometry collision mesh filename=package://voaige_description/arms/kinova_gen3/meshes/forear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; visual mesh filename=package://voaige_description/arms/kinova_gen3/meshes/forear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
- link shoulder_link: geometry collision mesh filename=package://voaige_description/arms/kinova_gen3/meshes/should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; visual mesh filename=package://voaige_description/arms/kinova_gen3/meshes/should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
- link sphericalwrist1_link: geometry collision mesh filename=package://voaige_description/arms/kinova_gen3/meshes/spheri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; visual mesh filename=package://voaige_description/arms/kinova_gen3/meshes/spheri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
- link sphericalwrist2_link: geometry collision mesh filename=package://voaige_description/arms/kinova_gen3/meshes/spheri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; visual mesh filename=package://voaige_description/arms/kinova_gen3/meshes/spheri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
